File: hw/puck_led/puck_led.kicad_sch (KiCad schematic)
At the start: 11 parts

Commit message: Added test mode
Parts:
- C1: LCSC (none) -> C307331; Supplier Part C307331 -> (none)
- LED1, LED2: LCSC (none) -> C396643; Supplier Part C396643 -> (none)
- Q1: LCSC (none) -> C2869182; Supplier Part C2869182 -> (none)
- R1: LCSC (none) -> C25741; Supplier Part C25741 -> (none)
- R2, R3: LCSC (none) -> C25082; Supplier Part C25082 -> (none)
- U1: LCSC (none) -> C2655038; Supplier Part C2655038 -> (none)
Changed lines of the file:
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@@
 			)
 		)
-		(property "Supplier Part" "C25082"
+		(property "LCSC" "C25082"
 			(at 130.81 53.34 0)
 			(hide yes)
@@
 			)
 		)
-		(property "Supplier Part" "C396643"
+		(property "LCSC" "C396643"
 			(at 116.84 63.5 0)
 			(hide yes)
@@
 			)
 		)
-		(property "Supplier Part" "C2655038"
+		(property "LCSC" "C2655038"
 			(at 83.82 58.42 0)
 			(hide yes)
@@
 			)
 		)
-		(property "Supplier Part" "C307331"
+		(property "LCSC" "C307331"
 			(at 57.15 63.5 0)
 			(hide yes)
@@
 			)
 		)
-		(property "Supplier Part" "C25741"
+		(property "LCSC" "C25741"
 			(at 91.44 78.74 0)
 			(hide yes)
@@
 			)
 		)
-		(property "Supplier Part" "C25082"
+		(property "LCSC" "C25082"
 			(at 116.84 53.34 0)
 			(hide yes)
@@
 			)
 		)
-		(property "Supplier Part" "C396643"
+		(property "LCSC" "C396643"
 			(at 130.81 63.5 0)
 			(hide yes)
@@
 			)
 		)
-		(property "Supplier Part" "C2869182"
+		(property "LCSC" "C2869182"
 			(at 116.84 73.66 0)
 			(hide yes)
